File: microNode/microNode.sch (EAGLE design)
At the start: 29 parts, among them U1 ATSAMD21G18A-AU, U2 TPL5111, U3 RFM95W-868S2, U4 MIC5504-3.3YM5-T5, U6 CLX6E-FKC-CH1M1D1BB7C3D3, U7 SIP32431DR3, U8 PCF2123, Y1 ABS07, Y2 ABS07

Commit message: Display connector/ RST button/ side led
Parts:
- removed U6: CLX6E-FKC-CH1M1D1BB7C3D3, CLX6E-FKC:CLX6E-FKC-CH1M1D1BB7C3D3
- added JP4: (no value), pinhead:PINHD-1X8
- added U$1: MSL0104RGB, MSL0104RGB:MSL0104RGB
- added U$2: KMR731NG, button:KMR731NG
- JP1: device pinhead:PINHD-1X4 -> pinhead:PINHD-1X5
Connections:
- removed net N$10: R5.2, U6.R-
- removed net N$7: R3.2, U6.B-
- removed net N$9: R4.2, U6.G-
- new net N$12: R3.1, U$1.R_A
- new net N$13: R4.1, U$1.G_A
- new net N$14: R5.1, U$1.B_A
- net 3V3: now also JP1.1, JP4.2
- net D11: now also R3.2; no longer U6.R+
- net D12: now also R4.2; no longer U6.G+
- net D13: now also R5.2; no longer U6.B+
- net D3: now also JP4.5
- net D4: now also JP4.6
- net D5: now also JP4.7
- net D6: now also JP4.8
- net GND: now also JP1.2, JP4.1, U$1.B_C, U$1.G_C, U$1.R_C, U$2.2; no longer JP1.1, R3.1, R4.1, R5.1
- net MOSI: now also JP4.3
- net RST: now also JP1.3, U$2.1; no longer JP1.2
- net SCK: now also JP4.4
- net SWCLK: now also JP1.4; no longer JP1.3
- net SWDIO: now also JP1.5; no longer JP1.4
Other:
- moved on the sheet: R3, R4, R5
