File: powersense_pcb/powersense.sch (EAGLE design)
At the start: 66 parts, among them IC1 ADG608R, IC2 LM741D, U1 LT1494CS8PBF, U2 LT1494CS8PBF, U3 LM77051, U4 BQ25504RGT, U5 SIP32431DR3, X1 1727036, X2 1727036, X3 1727036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

Commit message: changed coin cell holder
Parts:
- removed R16: PD1, rcl:R-EU_R0603
- removed R17: PD2, rcl:R-EU_R0603
- removed SJ3: (no value), jumper:SJ
- removed U$1: (no value), adafruit:CR2032SMT
- added BT1: (no value), SparkFun-Batteries:BATTERY-20MM_SMD
Connections:
- removed net N$11: R16.2, SJ3.2
- net A0: no longer J1.2
- net A4: now also J1.2; no longer R16.1, R17.2
- net GND: now also BT1.-; no longer R17.1, U$1.+, U$1.+1
- net JEFF: no longer SJ3.1
- net VRTC: now also BT1.+; no longer U$1.-
Changed lines of the file:
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@@
 <?xml version="1.0" encoding="utf-8"?>
 <!DOCTYPE eagle SYSTEM "eagle.dtd">
-<eagle version="9.0.1">
+<eagle version="9.1.2">
 <drawing>
 <settings>
@@
 <part name="J1" library="pinhead" library_urn="urn:adsk.eagle:library:325" deviceset="PINHD-1X5" device="" package3d_urn="urn:adsk.eagle:package:22469/2"/>
 <part name="VDD7" library="supply1" deviceset="VDD" device=""/>
-<part name="U$1" library="adafruit" deviceset="CR2032" device="SMT"/>
 <part name="U4" library="BQ25504" deviceset="BQ25504" device="RGT"/>
 <part name="R7" library="rcl" deviceset="R-EU_" device="R0603" value="OC2"/>
@@
 <part name="U5" library="SIP32431DR3T1GE3" deviceset="SIP32431DR3" device=""/>
 <part name="SJ2" library="jumper" deviceset="SJ" device=""/>
-<part name="SJ3" library="jumper" deviceset="SJ" device=""/>
 <part name="JP2" library="pinhead" library_urn="urn:adsk.eagle:library:325" deviceset="PINHD-1X2" device="" package3d_urn="urn:adsk.eagle:package:22435/2"/>
 <part name="SJ4" library="jumper" deviceset="SJ" device=""/>
-<part name="R16" library="rcl" deviceset="R-EU_" device="R0603" value="PD1"/>
-<part name="R17" library="rcl" deviceset="R-EU_" device="R0603" value="PD2"/>
 <part name="JP3" library="pinhead" library_urn="urn:adsk.eagle:library:325" deviceset="PINHD-1X2" device="" package3d_urn="urn:adsk.eagle:package:22435/2"/>
 <part name="SJ5" library="jumper" deviceset="SJ" device=""/>
 <part name="R18" library="rcl" deviceset="R-EU_" device="R0603" value="10M"/>
+<part name="BT1" library="SparkFun-Batteries" deviceset="BATTERY" device="-20MM_SMD"/>
 </parts>
 <sheets>
@@
 <instance part="J1" gate="A" x="-10.16" y="180.34" rot="MR0"/>
 <instance part="VDD7" gate="G$1" x="205.74" y="66.548"/>
-<instance part="U$1" gate="G$1" x="134.62" y="15.24"/>
 <instance part="U4" gate="G$1" x="172.72" y="121.92"/>
 <instance part="R7" gate="G$1" x="127" y="157.48" rot="R90"/>
@@
 <instance part="U5" gate="G$1" x="251.46" y="165.1"/>
 <instance part="SJ2" gate="1" x="109.22" y="187.96"/>
-<instance part="SJ3" gate="1" x="246.38" y="139.7"/>
 <instance part="JP2" gate="G$1" x="233.68" y="20.32" rot="R90"/>
 <instance part="SJ4" gate="1" x="233.68" y="5.08"/>
-<instance part="R16" gate="G$1" x="261.62" y="121.92" rot="R90"/>
-<instance part="R17" gate="G$1" x="261.62" y="106.68" rot="R90"/>
 <instance part="JP3" gate="G$1" x="231.14" y="63.5" rot="R90"/>
 <instance part="SJ5" gate="1" x="231.14" y="50.8"/>
 <instance part="R18" gate="G$1" x="104.14" y="149.86"/>
+<instance part="BT1" gate="G$1" x="134.62" y="15.24" rot="R180"/>
 </instances>
 <busses>
@@
 <wire x1="-7.62" y1="175.26" x2="15.24" y2="175.26" width="0.1524" layer="91"/>
 <label x="12.7" y="175.26" size="1.778" layer="95"/>
-</segment>
-<segment>
-<pinref part="U$1" gate="G$1" pin="+"/>
-<pinref part="U$1" gate="G$1" pin="+1"/>
-<wire x1="139.7" y1="17.78" x2="139.7" y2="12.7" width="0.1524" layer="91"/>
-<wire x1="139.7" y1="12.7" x2="152.4" y2="12.7" width="0.1524" layer="91"/>
-<junction x="139.7" y="12.7"/>
-<label x="147.32" y="12.7" size="1.778" layer="95"/>
 </segment>
 <segment>
@@
 <wire x1="83.82" y1="167.64" x2="83.82" y2="149.86" width="0.1524" layer="91"/>
 <wire x1="83.82" y1="149.86" x2="96.52" y2="149.86" width="0.1524" layer="91"/>
-<wire x1="238.76" y1="91.44" x2="261.62" y2="91.44" width="0.1524" layer="91"/>
-<wire x1="261.62" y1="91.44" x2="276.86" y2="91.44" width="0.1524" layer="91"/>
+<wire x1="238.76" y1="91.44" x2="276.86" y2="91.44" width="0.1524" layer="91"/>
 <wire x1="276.86" y1="91.44" x2="276.86" y2="149.86" width="0.1524" layer="91"/>
 <junction x="238.76" y="91.44"/>
@@
 <junction x="96.52" y="91.44"/>
 <label x="83.82" y="91.44" size="1.778" layer="95"/>
-<pinref part="R17" gate="G$1" pin="1"/>
-<wire x1="261.62" y1="101.6" x2="261.62" y2="91.44" width="0.1524" layer="91"/>
-<junction x="261.62" y="91.44"/>
 <pinref part="R18" gate="G$1" pin="1"/>
 <wire x1="96.52" y1="149.86" x2="99.06" y2="149.86" width="0.1524" layer="91" style="longdash"/>
+</segment>
+<segment>
+<wire x1="129.54" y1="15.24" x2="114.3" y2="15.24" width="0.1524" layer="91"/>
+<label x="114.3" y="15.24" size="1.778" layer="95"/>
+<pinref part="BT1" gate="G$1" pin="-"/>
 </segment>
 </net>
@@
 <label x="256.54" y="33.02" size="1.778" layer="95"/>
 </segment>
-<segment>
-<pinref part="J1" gate="A" pin="2"/>
-<wire x1="-7.62" y1="182.88" x2="15.24" y2="182.88" width="0.1524" layer="91"/>
-<label x="12.7" y="182.88" size="1.778" layer="95"/>
-</segment>
 </net>
 <net name="A1" class="0">
@@
 <wire x1="238.76" y1="121.92" x2="238.76" y2="139.7" width="0.1524" layer="91"/>
 <wire x1="238.76" y1="139.7" x2="195.58" y2="139.7" width="0.1524" layer="91"/>
-<pinref part="SJ3" gate="1" pin="1"/>
-<wire x1="241.3" y1="139.7" x2="238.76" y2="139.7" width="0.1524" layer="91"/>
-<junction x="238.76" y="139.7"/>
 </segment>
 </net>
@@
 </segment>
 <segment>
-<pinref part="U$1" gate="G$1" pin="-"/>
-<wire x1="129.54" y1="15.24" x2="114.3" y2="15.24" width="0.1524" layer="91"/>
-<label x="114.3" y="15.24" size="1.778" layer="95"/>
+<wire x1="139.7" y1="15.24" x2="157.48" y2="15.24" width="0.1524" layer="91"/>
+<label x="149.86" y="15.24" size="1.778" layer="95"/>
+<pinref part="BT1" gate="G$1" pin="+"/>
 </segment>
 </net>
@@
 </segment>
 <segment>
-<pinref part="R16" gate="G$1" pin="1"/>
-<pinref part="R17" gate="G$1" pin="2"/>
-<wire x1="261.62" y1="116.84" x2="261.62" y2="114.3" width="0.1524" layer="91"/>
-<wire x1="261.62" y1="114.3" x2="261.62" y2="111.76" width="0.1524" layer="91"/>
-<wire x1="261.62" y1="114.3" x2="269.24" y2="114.3" width="0.1524" layer="91"/>
-<junction x="261.62" y="114.3"/>
-<label x="264.16" y="114.3" size="1.778" layer="95"/>
+<pinref part="J1" gate="A" pin="2"/>
+<wire x1="-7.62" y1="182.88" x2="15.24" y2="182.88" width="0.1524" layer="91"/>
+<label x="12.7" y="182.88" size="1.778" layer="95"/>
 </segment>
 </net>
@@
 </segment>
 </net>
-<net name="N$11" class="0">
-<segment>
-<pinref part="SJ3" gate="1" pin="2"/>
-<pinref part="R16" gate="G$1" pin="2"/>
-<wire x1="251.46" y1="139.7" x2="261.62" y2="139.7" width="0.1524" layer="91"/>
-<wire x1="261.62" y1="139.7" x2="261.62" y2="127" width="0.1524" layer="91"/>
-</segment>
-</net>
